File: Kicad/80c51_memscan/80c51_memscan.sch (KiCad schematic (older format))
At the start: 18 parts, among them J1 Conn_02x16_Male, J2 Conn_01x02_Male, SW1 SW_SPST, U1 P80C51FA-4N,112, Y1 4-12Mhz

Commit message: Fixes and changes to needed to get the PCB going (change J1 symbol to match footprints. Mounting holes added to schematic to match PCB requirements, etc.
Parts:
- added MK1, MK10, MK11, MK12, MK2, MK3, MK4, MK5, MK6, MK7, MK8, MK9: MountingHole, MountingHole:MountingHole_8.4mm_M8, symbol Mechanical:MountingHole
- J1: symbol Connector_Generic:Conn_02x16_Counter_Clockwise -> Connector_Generic:Conn_02x16_Odd_Even
Connections:
- net A1: now also J1.3 (Pin_3); no longer J1.2 (Pin_2)
- net A10: now also J1.21 (Pin_21); no longer J1.11 (Pin_11)
- net A11: now also J1.23 (Pin_23); no longer J1.12 (Pin_12)
- net A2: now also J1.5 (Pin_5); no longer J1.3 (Pin_3)
- net A3: now also J1.7 (Pin_7); no longer J1.4 (Pin_4)
- net A4: now also J1.9 (Pin_9); no longer J1.5 (Pin_5)
- net A5: now also J1.11 (Pin_11); no longer J1.6 (Pin_6)
- net A6: now also J1.13 (Pin_13); no longer J1.7 (Pin_7)
- net A7: now also J1.15 (Pin_15); no longer J1.8 (Pin_8)
- net A8: now also J1.17 (Pin_17); no longer J1.9 (Pin_9)
- net A9: now also J1.19 (Pin_19); no longer J1.10 (Pin_10)
- net ALEn: now also J1.25 (Pin_25); no longer J1.13 (Pin_13)
- net Earth: now also J1.10 (Pin_10), J1.12 (Pin_12), J1.14 (Pin_14), J1.16 (Pin_16), J1.2 (Pin_2), J1.4 (Pin_4), J1.6 (Pin_6), J1.8 (Pin_8); no longer J1.17 (Pin_17), J1.19 (Pin_19), J1.21 (Pin_21), J1.23 (Pin_23), J1.25 (Pin_25), J1.27 (Pin_27), J1.29 (Pin_29), J1.31 (Pin_31)
- net PSENn: now also J1.27 (Pin_27); no longer J1.14 (Pin_14)
Changed lines of the file:
@@
 	2500 3600 3350 3600
 $Comp
-L Connector_Generic:Conn_02x16_Counter_Clockwise J1
+L Connector_Generic:Conn_02x16_Odd_Even J1
 U 1 1 5D6B2B27
 P 8700 5000
@@
 	0    -1   -1   0
 $EndComp
+$Comp
+L Mechanical:MountingHole MK1
+U 1 1 5D744743
+P 950 6550
+F 0 "MK1" H 1050 6596 50  0000 L CNN
+F 1 "MountingHole" H 1050 6505 50  0000 L CNN
+F 2 "MountingHole:MountingHole_8.4mm_M8" H 950 6550 50  0001 C CNN
+F 3 "~" H 950 6550 50  0001 C CNN
+	1    950  6550
+	1    0    0    -1
+$EndComp
+$Comp
+L Mechanical:MountingHole MK5
+U 1 1 5D7449F9
+P 1850 6550
+F 0 "MK5" H 1950 6596 50  0000 L CNN
+F 1 "MountingHole" H 1950 6505 50  0000 L CNN
+F 2 "MountingHole:MountingHole_8.4mm_M8" H 1850 6550 50  0001 C CNN
+F 3 "~" H 1850 6550 50  0001 C CNN
+	1    1850 6550
+	1    0    0    -1
+$EndComp
+$Comp
+L Mechanical:MountingHole MK9
+U 1 1 5D744A55
+P 2750 6550
+F 0 "MK9" H 2850 6596 50  0000 L CNN
+F 1 "MountingHole" H 2850 6505 50  0000 L CNN
+F 2 "MountingHole:MountingHole_8.4mm_M8" H 2750 6550 50  0001 C CNN
+F 3 "~" H 2750 6550 50  0001 C CNN
+	1    2750 6550
+	1    0    0    -1
+$EndComp
+$Comp
+L Mechanical:MountingHole MK2
+U 1 1 5D744AAF
+P 950 6850
+F 0 "MK2" H 1050 6896 50  0000 L CNN
+F 1 "MountingHole" H 1050 6805 50  0000 L CNN
+F 2 "MountingHole:MountingHole_8.4mm_M8" H 950 6850 50  0001 C CNN
+F 3 "~" H 950 6850 50  0001 C CNN
+	1    950  6850
+	1    0    0    -1
+$EndComp
+$Comp
+L Mechanical:MountingHole MK6
+U 1 1 5D744B2D
+P 1850 6850
+F 0 "MK6" H 1950 6896 50  0000 L CNN
+F 1 "MountingHole" H 1950 6805 50  0000 L CNN
+F 2 "MountingHole:MountingHole_8.4mm_M8" H 1850 6850 50  0001 C CNN
+F 3 "~" H 1850 6850 50  0001 C CNN
+	1    1850 6850
+	1    0    0    -1
+$EndComp
+$Comp
+L Mechanical:MountingHole MK10
+U 1 1 5D744B8D
+P 2750 6850
+F 0 "MK10" H 2850 6896 50  0000 L CNN
+F 1 "MountingHole" H 2850 6805 50  0000 L CNN
+F 2 "MountingHole:MountingHole_8.4mm_M8" H 2750 6850 50  0001 C CNN
+F 3 "~" H 2750 6850 50  0001 C CNN
+	1    2750 6850
+	1    0    0    -1
+$EndComp
+$Comp
+L Mechanical:MountingHole MK3
+U 1 1 5D744BF7
+P 950 7150
+F 0 "MK3" H 1050 7196 50  0000 L CNN
+F 1 "MountingHole" H 1050 7105 50  0000 L CNN
+F 2 "MountingHole:MountingHole_8.4mm_M8" H 950 7150 50  0001 C CNN
+F 3 "~" H 950 7150 50  0001 C CNN
+	1    950  7150
+	1    0    0    -1
+$EndComp
+$Comp
+L Mechanical:MountingHole MK7
+U 1 1 5D744C4D
+P 1850 7150
+F 0 "MK7" H 1950 7196 50  0000 L CNN
+F 1 "MountingHole" H 1950 7105 50  0000 L CNN
+F 2 "MountingHole:MountingHole_8.4mm_M8" H 1850 7150 50  0001 C CNN
+F 3 "~" H 1850 7150 50  0001 C CNN
+	1    1850 7150
+	1    0    0    -1
+$EndComp
+$Comp
+L Mechanical:MountingHole MK11
+U 1 1 5D744CB1
+P 2750 7150
+F 0 "MK11" H 2850 7196 50  0000 L CNN
+F 1 "MountingHole" H 2850 7105 50  0000 L CNN
+F 2 "MountingHole:MountingHole_8.4mm_M8" H 2750 7150 50  0001 C CNN
+F 3 "~" H 2750 7150 50  0001 C CNN
+	1    2750 7150
+	1    0    0    -1
+$EndComp
+$Comp
+L Mechanical:MountingHole MK4
+U 1 1 5D74DDA9
+P 950 7450
+F 0 "MK4" H 1050 7496 50  0000 L CNN
+F 1 "MountingHole" H 1050 7405 50  0000 L CNN
+F 2 "MountingHole:MountingHole_8.4mm_M8" H 950 7450 50  0001 C CNN
+F 3 "~" H 950 7450 50  0001 C CNN
+	1    950  7450
+	1    0    0    -1
+$EndComp
+$Comp
+L Mechanical:MountingHole MK8
+U 1 1 5D74DE07
+P 1850 7450
+F 0 "MK8" H 1950 7496 50  0000 L CNN
+F 1 "MountingHole" H 1950 7405 50  0000 L CNN
+F 2 "MountingHole:MountingHole_8.4mm_M8" H 1850 7450 50  0001 C CNN
+F 3 "~" H 1850 7450 50  0001 C CNN
+	1    1850 7450
+	1    0    0    -1
+$EndComp
+$Comp
+L Mechanical:MountingHole MK12
+U 1 1 5D74DEA3
+P 2750 7450
+F 0 "MK12" H 2850 7496 50  0000 L CNN
+F 1 "MountingHole" H 2850 7405 50  0000 L CNN
+F 2 "MountingHole:MountingHole_8.4mm_M8" H 2750 7450 50  0001 C CNN
+F 3 "~" H 2750 7450 50  0001 C CNN
+	1    2750 7450
+	1    0    0    -1
+$EndComp
 $EndSCHEMATC

Commit message: Initial PCB layout complete.
Parts:
- D1: footprint LED_SMD:LED_0603_1608Metric -> LED_SMD:LED_0603_1608Metric_Pad1.05x0.95mm_HandSolder
- J2: footprint Connector_PinHeader_2.54mm:PinHeader_1x02_P2.54mm_Vertical -> Connector_Molex:Molex_KK-254_AE-6410-02A_1x02_P2.54mm_Vertical
Changed lines of the file:
@@
 F 0 "J2" H 2008 1531 50  0000 C CNN
 F 1 "Conn_01x02_Male" H 2008 1440 50  0000 C CNN
-F 2 "Connector_PinHeader_2.54mm:PinHeader_1x02_P2.54mm_Vertical" H 1900 1350 50  0001 C CNN
+F 2 "Connector_Molex:Molex_KK-254_AE-6410-02A_1x02_P2.54mm_Vertical" H 1900 1350 50  0001 C CNN
 F 3 "~" H 1900 1350 50  0001 C CNN
 	1    1900 1350
@@
 F 0 "D1" H 3192 1095 50  0000 C CNN
 F 1 "LED" H 3192 1186 50  0000 C CNN
-F 2 "LED_SMD:LED_0603_1608Metric" H 3200 1350 50  0001 C CNN
+F 2 "LED_SMD:LED_0603_1608Metric_Pad1.05x0.95mm_HandSolder" H 3200 1350 50  0001 C CNN
 F 3 "~" H 3200 1350 50  0001 C CNN
 	1    3200 1350
